Commit message: added the joint_state_controller

File: install/ugv/share/ugv/urdf/ugv1.xacro (robot description, xacro)
@@ -1,7 +1,8 @@
 <?xml version="1.0"?>
 <robot xmlns:xacro="http://www.ros.org/wiki/xacro" name="ugv">
-<xacro:property name="mainBody" value= "package://ugv/mesh//mainBody.obj"/>
-<xacro:property name="wheel" value= "package://ugv/mesh/tyre.obj"/>
-<xacro:property name="lidar" value= "package://ugv/mesh/lidar.obj"/>
+<xacro:property name="mainBody" value= "file:///home/david/urdf_tutorial/obj/mainBody.obj"/>
+<xacro:property name="wheel" value= "file:///home/david/urdf_tutorial/obj/tyre.obj"/>
+<xacro:property name="lidar" value= "file:///home/david/urdf_tutorial/obj/lidar.obj"/>
+<xacro:property name="shaft" value= "file:///home/david/urdf_tutorial/obj/shaft.obj"/>
 <xacro:property name="scale" value = "1 1 1"/>
 <xacro:macro name="wheel" params="name">
@@ -44,23 +45,59 @@
     </visual>
 </link>
-<joint name="mainBody_WheelBL" type="fixed">
+<link name="shaftF">
+    <visual>
+        <origin xyz="0.0 0.0 0.0" rpy="1.57 0.0 0.0"/>
+        <geometry>
+            <mesh filename="${shaft}" scale= "${scale}"/>
+        </geometry>
+        <material name="grey"/>
+    </visual>
+</link>
+<link name="shaftB">
+    <visual>
+        <origin xyz="0.0 0.0 0.0" rpy="1.57 0.0 0.0"/>
+        <geometry>
+            <mesh filename="${shaft}" scale= "${scale}"/>
+        </geometry>
+        <material name="grey"/>
+    </visual>
+</link>
+<joint name="mainBody_shaftF" type="fixed">
+    <parent link="base_link"/>
+    <child link="shaftF"/>
+    <origin xyz="0.07 0 0.0105" rpy="0.0 0.0 0.0"/>
+</joint>
+<joint name="mainBody_shaftB" type="fixed">
+    <parent link="base_link"/>
+    <child link="shaftB"/>
+    <origin xyz="-0.07 0 0.0105" rpy="0.0 0.0 0.0"/>
+</joint>
+<joint name="mainBody_WheelBL" type="continuous">
     <parent link="base_link"/>
     <child link="wheelBL"/>
     <origin xyz="-0.07 0.0525 0.01" rpy="0.0 0.0 0.0"/>
+    <axis xyz="0 1 0"/>
+    <limit lower="0" upper="0" effort="0" velocity="0"/>
 </joint>
-<joint name="mainBody_WheelFL" type="fixed">
+<joint name="mainBody_WheelFL" type="continuous">
     <parent link="base_link"/>
     <child link="wheelFL"/>
     <origin xyz="0.07 0.0525 0.010" rpy="0.0 0.0 0.0"/>
+    <axis xyz="0 1 0"/>
+    <limit lower="0" upper="0" effort="0" velocity="0"/>
 </joint>
-<joint name="mainBody_WheelFR" type="fixed">
+<joint name="mainBody_WheelFR" type="continuous">
     <parent link="base_link"/>
     <child link="wheelFR"/>
     <origin xyz="0.07 -0.0525 0.010" rpy="0.0 0.0 0.0"/>
+    <axis xyz="0 1 0"/>
+    <limit lower="0" upper="0" effort="0" velocity="0"/>
 </joint>
-<joint name="mainBody_WheelBR" type="fixed">
+<joint name="mainBody_WheelBR" type="continuous">
     <parent link="base_link"/>
     <child link="wheelBR"/>
     <origin xyz="-0.07 -0.0525 0.010" rpy="0.0 0.0 0.0"/>
+    <axis xyz="0 1 0"/>
+    <limit lower="0" upper="0" effort="0" velocity="0"/>
 </joint>
 <joint name="mainBody_Lidar" type="fixed">
