Commit message: M2

File: install/ugv/share/ugv/urdf/ugv.xacro (robot description, xacro)
@@ -3,5 +3,5 @@
 <xacro:property name="mainBody" value= "package://ugv/mesh/mainBodyv2.obj"/>
 <xacro:property name="wheel" value= "package://ugv/mesh/tyrev2.obj"/>
-<xacro:property name="scale" value = "0.01 0.01 0.01"/>
+<xacro:property name="scale" value = "0.1 0.1 0.1"/>
 <xacro:macro name="wheel" params="name">
     <link name="${name}">
@@ -37,5 +37,5 @@
     <parent link="base_link"/>
     <child link="wheelBL"/>
-    <origin xyz="-0.07 0.057 0.010" rpy="0.0 0.0 0.0"/>
+    <origin xyz="-0.7 0.57 0.10" rpy="0.0 0.0 0.0"/>
 </joint>
 <joint name="mainBody_WheelFL" type="fixed">

File: src/ugv/urdf/ugv1.xacro (robot description, xacro)
@@ -1,11 +1,12 @@
 <?xml version="1.0"?>
 <robot xmlns:xacro="http://www.ros.org/wiki/xacro" name="ugv">
-<xacro:property name="mainBody" value= "package://ugv/mesh/mainBodyv2.obj"/>
-<xacro:property name="wheel" value= "package://ugv/mesh/tyrev2.obj"/>
-<xacro:property name="scale" value = "0.1 0.1 0.1"/>
+<xacro:property name="mainBody" value= "package://ugv/mesh//mainBody.obj"/>
+<xacro:property name="wheel" value= "package://ugv/mesh/tyre.obj"/>
+<xacro:property name="lidar" value= "package://ugv/mesh/lidar.obj"/>
+<xacro:property name="scale" value = "1 1 1"/>
 <xacro:macro name="wheel" params="name">
     <link name="${name}">
     <visual>
-        <origin xyz="0.0 0.0 0.0" rpy="0.0 0.0 0.0"/>
+        <origin xyz="0.0 0.0 0.0" rpy="1.57 0.0 0.0"/>
         <geometry>
             <mesh filename="${wheel}" scale="${scale}"/>
@@ -27,7 +28,16 @@
 <link name="base_link">
     <visual>
-        <origin xyz="0.0 0.0 0.0" rpy="0.0 0.0 0.0"/>
+        <origin xyz="0.0 0.0 0.0" rpy="1.57 0.0 0.0"/>
         <geometry>
             <mesh filename="${mainBody}" scale= "${scale}"/>
+        </geometry>
+        <material name="grey"/>
+    </visual>
+</link>
+<link name="lidar">
+    <visual>
+        <origin xyz="0.0 0.0 0.0" rpy="1.57 0.0 0.0"/>
+        <geometry>
+            <mesh filename="${lidar}" scale= "${scale}"/>
         </geometry>
         <material name="grey"/>
@@ -37,20 +47,25 @@
     <parent link="base_link"/>
     <child link="wheelBL"/>
-    <origin xyz="-0.7 0.57 0.10" rpy="0.0 0.0 0.0"/>
+    <origin xyz="-0.07 0.0525 0.01" rpy="0.0 0.0 0.0"/>
 </joint>
 <joint name="mainBody_WheelFL" type="fixed">
     <parent link="base_link"/>
     <child link="wheelFL"/>
-    <origin xyz="0.07 0.057 0.010" rpy="0.0 0.0 0.0"/>
+    <origin xyz="0.07 0.0525 0.010" rpy="0.0 0.0 0.0"/>
 </joint>
 <joint name="mainBody_WheelFR" type="fixed">
     <parent link="base_link"/>
     <child link="wheelFR"/>
-    <origin xyz="0.07 -0.048 0.010" rpy="0.0 0.0 0.0"/>
+    <origin xyz="0.07 -0.0525 0.010" rpy="0.0 0.0 0.0"/>
 </joint>
 <joint name="mainBody_WheelBR" type="fixed">
     <parent link="base_link"/>
     <child link="wheelBR"/>
-    <origin xyz="-0.07 -0.048 0.010" rpy="0.0 0.0 0.0"/>
+    <origin xyz="-0.07 -0.0525 0.010" rpy="0.0 0.0 0.0"/>
+</joint>
+<joint name="mainBody_Lidar" type="fixed">
+    <parent link="base_link"/>
+    <child link="lidar"/>
+    <origin xyz="0.075 0 0.04" rpy="0.0 0.0 0.0"/>
 </joint>
 </robot>

Commit message: updatedV1

File: install/ugv/share/ugv/urdf/ugv.xacro (robot description, xacro)
@@ -1,11 +1,13 @@
 <?xml version="1.0"?>
 <robot xmlns:xacro="http://www.ros.org/wiki/xacro" name="ugv">
-<xacro:property name="mainBody" value= "package://ugv/mesh/mainBodyv2.obj"/>
-<xacro:property name="wheel" value= "package://ugv/mesh/tyrev2.obj"/>
-<xacro:property name="scale" value = "0.1 0.1 0.1"/>
+<xacro:property name="mainBody" value= "package://ugv/mesh/mainBody.obj"/>
+<xacro:property name="wheel" value= "package://ugv/mesh/tyre.obj"/>
+<xacro:property name="lidar" value= "package://ugv/mesh/lidar.obj"/>
+<xacro:property name="shaft" value= "package://ugv/mesh/shaft.obj"/>
+<xacro:property name="scale" value = "1 1 1"/>
 <xacro:macro name="wheel" params="name">
     <link name="${name}">
     <visual>
-        <origin xyz="0.0 0.0 0.0" rpy="0.0 0.0 0.0"/>
+        <origin xyz="0.0 0.0 0.0" rpy="1.57 0.0 0.0"/>
         <geometry>
             <mesh filename="${wheel}" scale="${scale}"/>
@@ -27,5 +29,5 @@
 <link name="base_link">
     <visual>
-        <origin xyz="0.0 0.0 0.0" rpy="0.0 0.0 0.0"/>
+        <origin xyz="0.0 0.0 0.009" rpy="1.57 0.0 0.0"/>
         <geometry>
             <mesh filename="${mainBody}" scale= "${scale}"/>
@@ -34,23 +36,73 @@
     </visual>
 </link>
-<joint name="mainBody_WheelBL" type="fixed">
+<link name="lidar">
+    <visual>
+        <origin xyz="0.0 0.0 0.009" rpy="1.57 0.0 0.0"/>
+        <geometry>
+            <mesh filename="${lidar}" scale= "${scale}"/>
+        </geometry>
+        <material name="grey"/>
+    </visual>
+</link>
+<link name="shaftF">
+    <visual>
+        <origin xyz="0.0 0.0 0.009" rpy="1.57 0.0 0.0"/>
+        <geometry>
+            <mesh filename="${shaft}" scale= "${scale}"/>
+        </geometry>
+        <material name="grey"/>
+    </visual>
+</link>
+<link name="shaftB">
+    <visual>
+        <origin xyz="0.0 0.0 0.009" rpy="1.57 0.0 0.0"/>
+        <geometry>
+            <mesh filename="${shaft}" scale= "${scale}"/>
+        </geometry>
+        <material name="grey"/>
+    </visual>
+</link>
+<joint name="mainBody_shaftF" type="fixed">
+    <parent link="base_link"/>
+    <child link="shaftF"/>
+    <origin xyz="0.07 0 0.0105" rpy="0.0 0.0 0.0"/>
+</joint>
+<joint name="mainBody_shaftB" type="fixed">
+    <parent link="base_link"/>
+    <child link="shaftB"/>
+    <origin xyz="-0.07 0 0.0105" rpy="0.0 0.0 0.0"/>
+</joint>
+<joint name="mainBody_WheelBL" type="continuous">
     <parent link="base_link"/>
     <child link="wheelBL"/>
-    <origin xyz="-0.7 0.57 0.10" rpy="0.0 0.0 0.0"/>
+    <origin xyz="-0.07 0.0525 0.019" rpy="0.0 0.0 0.0"/>
+    <axis xyz="0 1 0"/>
+    <limit lower="0" upper="0" effort="0" velocity="0"/>
 </joint>
-<joint name="mainBody_WheelFL" type="fixed">
+<joint name="mainBody_WheelFL" type="continuous">
     <parent link="base_link"/>
     <child link="wheelFL"/>
-    <origin xyz="0.07 0.057 0.010" rpy="0.0 0.0 0.0"/>
+    <origin xyz="0.07 0.0525 0.019" rpy="0.0 0.0 0.0"/>
+    <axis xyz="0 1 0"/>
+    <limit lower="0" upper="0" effort="0" velocity="0"/>
 </joint>
-<joint name="mainBody_WheelFR" type="fixed">
+<joint name="mainBody_WheelFR" type="continuous">
     <parent link="base_link"/>
     <child link="wheelFR"/>
-    <origin xyz="0.07 -0.048 0.010" rpy="0.0 0.0 0.0"/>
+    <origin xyz="0.07 -0.0525 0.019" rpy="0.0 0.0 0.0"/>
+    <axis xyz="0 1 0"/>
+    <limit lower="0" upper="0" effort="0" velocity="0"/>
 </joint>
-<joint name="mainBody_WheelBR" type="fixed">
+<joint name="mainBody_WheelBR" type="continuous">
     <parent link="base_link"/>
     <child link="wheelBR"/>
-    <origin xyz="-0.07 -0.048 0.010" rpy="0.0 0.0 0.0"/>
+    <origin xyz="-0.07 -0.0525 0.019" rpy="0.0 0.0 0.0"/>
+    <axis xyz="0 1 0"/>
+    <limit lower="0" upper="0" effort="0" velocity="0"/>
+</joint>
+<joint name="mainBody_Lidar" type="fixed">
+    <parent link="base_link"/>
+    <child link="lidar"/>
+    <origin xyz="0.075 0 0.04" rpy="0.0 0.0 0.0"/>
 </joint>
 </robot>

File: src/ugv/urdf/ugv.xacro (robot description, xacro)
@@ -9,5 +9,5 @@
     <link name="${name}">
     <visual>
-        <origin xyz="0.0 0.0 0.009" rpy="1.57 0.0 0.0"/>
+        <origin xyz="0.0 0.0 0.0" rpy="1.57 0.0 0.0"/>
         <geometry>
             <mesh filename="${wheel}" scale="${scale}"/>
@@ -73,29 +73,29 @@
     <origin xyz="-0.07 0 0.0105" rpy="0.0 0.0 0.0"/>
 </joint>
-<joint name="mainBody_WheelBL" type="fixed">
+<joint name="mainBody_WheelBL" type="continuous">
     <parent link="base_link"/>
     <child link="wheelBL"/>
-    <origin xyz="-0.07 0.0525 0.01" rpy="0.0 0.0 0.0"/>
+    <origin xyz="-0.07 0.0525 0.019" rpy="0.0 0.0 0.0"/>
     <axis xyz="0 1 0"/>
     <limit lower="0" upper="0" effort="0" velocity="0"/>
 </joint>
-<joint name="mainBody_WheelFL" type="fixed">
+<joint name="mainBody_WheelFL" type="continuous">
     <parent link="base_link"/>
     <child link="wheelFL"/>
-    <origin xyz="0.07 0.0525 0.010" rpy="0.0 0.0 0.0"/>
+    <origin xyz="0.07 0.0525 0.019" rpy="0.0 0.0 0.0"/>
     <axis xyz="0 1 0"/>
     <limit lower="0" upper="0" effort="0" velocity="0"/>
 </joint>
-<joint name="mainBody_WheelFR" type="fixed">
+<joint name="mainBody_WheelFR" type="continuous">
     <parent link="base_link"/>
     <child link="wheelFR"/>
-    <origin xyz="0.07 -0.0525 0.010" rpy="0.0 0.0 0.0"/>
+    <origin xyz="0.07 -0.0525 0.019" rpy="0.0 0.0 0.0"/>
     <axis xyz="0 1 0"/>
     <limit lower="0" upper="0" effort="0" velocity="0"/>
 </joint>
-<joint name="mainBody_WheelBR" type="fixed">
+<joint name="mainBody_WheelBR" type="continuous">
     <parent link="base_link"/>
     <child link="wheelBR"/>
-    <origin xyz="-0.07 -0.0525 0.010" rpy="0.0 0.0 0.0"/>
+    <origin xyz="-0.07 -0.0525 0.019" rpy="0.0 0.0 0.0"/>
     <axis xyz="0 1 0"/>
     <limit lower="0" upper="0" effort="0" velocity="0"/>

Commit message: update_141124

File: install/ugv/share/ugv/urdf/ugv.xacro (robot description, xacro)
@@ -8,4 +8,9 @@
 <xacro:macro name="wheel" params="name">
     <link name="${name}">
+        <inertial>
+            <mass value="1.0"/>
+            <origin xyz="0 0 0"/>
+            <inertia ixx="0.01" iyy="0.01" izz="0.01" ixy="0" ixz="0" iyz="0"/>
+        </inertial>
     <visual>
         <origin xyz="0.0 0.0 0.0" rpy="1.57 0.0 0.0"/>
@@ -28,4 +33,9 @@
 </material>
 <link name="base_link">
+    <inertial>
+            <mass value="1.0"/>
+            <origin xyz="0 0 0"/>
+            <inertia ixx="0.01" iyy="0.01" izz="0.01" ixy="0" ixz="0" iyz="0"/>
+    </inertial>
     <visual>
         <origin xyz="0.0 0.0 0.009" rpy="1.57 0.0 0.0"/>
@@ -37,4 +47,9 @@
 </link>
 <link name="lidar">
+    <inertial>
+            <mass value="1.0"/>
+            <origin xyz="0 0 0"/>
+            <inertia ixx="0.01" iyy="0.01" izz="0.01" ixy="0" ixz="0" iyz="0"/>
+    </inertial>
     <visual>
         <origin xyz="0.0 0.0 0.009" rpy="1.57 0.0 0.0"/>
@@ -46,4 +61,9 @@
 </link>
 <link name="shaftF">
+    <inertial>
+            <mass value="1.0"/>
+            <origin xyz="0 0 0"/>
+            <inertia ixx="0.01" iyy="0.01" izz="0.01" ixy="0" ixz="0" iyz="0"/>
+    </inertial>
     <visual>
         <origin xyz="0.0 0.0 0.009" rpy="1.57 0.0 0.0"/>
@@ -55,4 +75,9 @@
 </link>
 <link name="shaftB">
+    <inertial>
+            <mass value="1.0"/>
+            <origin xyz="0 0 0"/>
+            <inertia ixx="0.01" iyy="0.01" izz="0.01" ixy="0" ixz="0" iyz="0"/>
+    </inertial>
     <visual>
         <origin xyz="0.0 0.0 0.009" rpy="1.57 0.0 0.0"/>
