Commit message: updated stl file

File: install/ugv/share/ugv/urdf/ugv.urdf (robot description, URDF)
Before this commit: robot ugv, 8 links, 7 joints
Links:
- link base_link: geometry visual mesh filename=package://ugv/mesh/mainBody.stl scale=1 1 1
- link lidar: geometry visual mesh filename=package://ugv/mesh/lidar.stl scale=1 1 1
- link shaftB: geometry visual mesh filename=package://ugv/mesh/shaft.stl scale=1 1 1
- link shaftF: geometry visual mesh filename=package://ugv/mesh/shaft.stl scale=1 1 1
- link wheelBL: geometry visual mesh filename=package://ugv/mesh/tyre.stl scale=1 1 1
- link wheelBR: geometry visual mesh filename=package://ugv/mesh/tyre.stl scale=1 1 1
- link wheelFL: geometry visual mesh filename=package://ugv/mesh/tyre.stl scale=1 1 1
- link wheelFR: geometry visual mesh filename=package://ugv/mesh/tyre.stl scale=1 1 1

File: install/ugv/share/ugv/urdf/ugvGazebo.xacro (robot description, xacro)
@@ -1,8 +1,8 @@
 <?xml version="1.0"?>
 <robot xmlns:xacro="http://www.ros.org/wiki/xacro" name="ugv">
-<xacro:property name="mainBody" value= "package://ugv/mesh/mainBody.obj"/>
-<xacro:property name="wheel" value= "package://ugv/mesh/tyre.obj"/>
-<xacro:property name="lidar" value= "package://ugv/mesh/lidar.obj"/>
-<xacro:property name="shaft" value= "package://ugv/mesh/shaft.obj"/>
+<xacro:property name="mainBody" value= "package://ugv/mesh/mainBody.stl"/>
+<xacro:property name="wheel" value= "package://ugv/mesh/tyre.stl"/>
+<xacro:property name="lidar" value= "package://ugv/mesh/lidar.stl"/>
+<xacro:property name="shaft" value= "package://ugv/mesh/shaft.stl"/>
 <xacro:property name="scale" value = "1 1 1"/>
 <xacro:macro name="wheel" params="name">

File: src/ugv/urdf/ugv1.xacro (robot description, xacro)
@@ -1,8 +1,8 @@
 <?xml version="1.0"?>
 <robot xmlns:xacro="http://www.ros.org/wiki/xacro" name="ugv">
-<xacro:property name="mainBody" value= "package://ugv/mesh/mainBody.obj"/>
-<xacro:property name="wheel" value= "package://ugv/mesh/tyre.obj"/>
-<xacro:property name="lidar" value= "package://ugv/mesh/lidar.obj"/>
-<xacro:property name="shaft" value= "package://ugv/mesh/shaft.obj"/>
+<xacro:property name="mainBody" value= "package://ugv/mesh/mainBody.stl"/>
+<xacro:property name="wheel" value= "package://ugv/mesh/tyre.stl"/>
+<xacro:property name="lidar" value= "package://ugv/mesh/lidar.stl"/>
+<xacro:property name="shaft" value= "package://ugv/mesh/shaft.stl"/>
 <xacro:property name="scale" value = "1 1 1"/>
 <xacro:macro name="wheel" params="name">

Commit message: updatedlater

File: install/ugv/share/ugv/urdf/ugv.urdf (robot description, URDF)
Before this commit: robot r2d2, 4 links, 3 joints
Links:
- removed link head
- removed link left_leg
- removed link right_leg
- added link lidar, mass 1.0; visual mesh filename=package://ugv/mesh/lidar.obj scale=1 1 1
- added link shaftB, mass 1.0; visual mesh filename=package://ugv/mesh/shaft.obj scale=1 1 1
- added link shaftF, mass 1.0; visual mesh filename=package://ugv/mesh/shaft.obj scale=1 1 1
- added link wheelBL, mass 1.0; visual mesh filename=package://ugv/mesh/tyre.obj scale=1 1 1
- added link wheelBR, mass 1.0; visual mesh filename=package://ugv/mesh/tyre.obj scale=1 1 1
- added link wheelFL, mass 1.0; visual mesh filename=package://ugv/mesh/tyre.obj scale=1 1 1
- added link wheelFR, mass 1.0; visual mesh filename=package://ugv/mesh/tyre.obj scale=1 1 1
- link base_link: mass 5.0 -> 1.0; geometry visual mesh filename=package://ugv/mesh/mainBody.obj scale=1 1 1
Joints:
- removed joint head_joint
- removed joint left_leg_joint
- removed joint right_leg_joint
- added joint mainBody_Lidar: type fixed, parent base_link, child lidar, origin xyz=0.075 0 0.04 rpy=0.0 0.0 0.0
- added joint mainBody_WheelBL: type continuous, parent base_link, child wheelBL, origin xyz=-0.07 0.0525 0.019 rpy=0.0 0.0 0.0, axis 0 1 0, limit lower=0 upper=0 effort=0 velocity=0
- added joint mainBody_WheelBR: type continuous, parent base_link, child wheelBR, origin xyz=-0.07 -0.0525 0.019 rpy=0.0 0.0 0.0, axis 0 1 0, limit lower=0 upper=0 effort=0 velocity=0
- added joint mainBody_WheelFL: type continuous, parent base_link, child wheelFL, origin xyz=0.07 0.0525 0.019 rpy=0.0 0.0 0.0, axis 0 1 0, limit lower=0 upper=0 effort=0 velocity=0
- added joint mainBody_WheelFR: type continuous, parent base_link, child wheelFR, origin xyz=0.07 -0.0525 0.019 rpy=0.0 0.0 0.0, axis 0 1 0, limit lower=0 upper=0 effort=0 velocity=0
- added joint mainBody_shaftB: type fixed, parent base_link, child shaftB, origin xyz=-0.07 0 0.0105 rpy=0.0 0.0 0.0
- added joint mainBody_shaftF: type fixed, parent base_link, child shaftF, origin xyz=0.07 0 0.0105 rpy=0.0 0.0 0.0

File: install/ugv/share/ugv/urdf/ugv.xacro (robot description, xacro)
@@ -1,3 +1,2 @@
-<?xml version="1.0"?>
 <robot xmlns:xacro="http://www.ros.org/wiki/xacro" name="ugv">
 <xacro:property name="mainBody" value= "package://ugv/mesh/mainBody.obj"/>
