Commit message: jetson

File: src/ugv/urdf/ugv.urdf (robot description, URDF)
Before this commit: robot ugv, 8 links, 7 joints
Links:
- removed link lidar
- removed link shaftB
- removed link shaftF
- removed link wheelBL
- removed link wheelBR
- removed link wheelFL
- removed link wheelFR
- added link head, mass 1.0; collision sphere radius=0.2; visual sphere radius=0.2
- added link left_leg, mass 1.0; collision box size=0.1 0.2 0.5; visual box size=0.1 0.2 0.5
- added link right_leg, mass 1.0; collision box size=0.1 0.2 0.5; visual box size=0.1 0.2 0.5
- link base_link: mass 0.2 -> 5.0; geometry collision cylinder length=0.6 radius=0.3; visual cylinder length=0.6 radius=0.3
Joints:
- removed joint mainBody_Lidar
- removed joint mainBody_WheelBL
- removed joint mainBody_WheelBR
- removed joint mainBody_WheelFL
- removed joint mainBody_WheelFR
- removed joint mainBody_shaftB
- removed joint mainBody_shaftF
- added joint head_joint: type fixed, parent base_link, child head, origin xyz=0 0 0.5 rpy=0 0 0
- added joint left_leg_joint: type fixed, parent base_link, child left_leg, origin xyz=0.25 0.2 0 rpy=0 0 0
- added joint right_leg_joint: type fixed, parent base_link, child right_leg, origin xyz=0.25 -0.2 0 rpy=0 0 0

File: src/ugv/urdf/ugv.xacro (robot description, xacro)
@@ -1,11 +1,13 @@
 <?xml version="1.0"?>
 <robot xmlns:xacro="http://www.ros.org/wiki/xacro" name="ugv">
-<xacro:property name="mainBody" value= "package://ugv/mesh/mainBodyv2.obj"/>
-<xacro:property name="wheel" value= "package://ugv/mesh/tyrev2.obj"/>
-<xacro:property name="scale" value = "0.1 0.1 0.1"/>
+<xacro:property name="mainBody" value= "package://ugv/mesh/mainBody.obj"/>
+<xacro:property name="wheel" value= "package://ugv/mesh/tyre.obj"/>
+<xacro:property name="lidar" value= "package://ugv/mesh/lidar.obj"/>
+<xacro:property name="shaft" value= "package://ugv/mesh/shaft.obj"/>
+<xacro:property name="scale" value = "1 1 1"/>
 <xacro:macro name="wheel" params="name">
     <link name="${name}">
     <visual>
-        <origin xyz="0.0 0.0 0.0" rpy="0.0 0.0 0.0"/>
+        <origin xyz="0.0 0.0 0.009" rpy="1.57 0.0 0.0"/>
         <geometry>
             <mesh filename="${wheel}" scale="${scale}"/>
@@ -27,5 +29,5 @@
 <link name="base_link">
     <visual>
-        <origin xyz="0.0 0.0 0.0" rpy="0.0 0.0 0.0"/>
+        <origin xyz="0.0 0.0 0.009" rpy="1.57 0.0 0.0"/>
         <geometry>
             <mesh filename="${mainBody}" scale= "${scale}"/>
@@ -34,23 +36,73 @@
     </visual>
 </link>
+<link name="lidar">
+    <visual>
+        <origin xyz="0.0 0.0 0.009" rpy="1.57 0.0 0.0"/>
+        <geometry>
+            <mesh filename="${lidar}" scale= "${scale}"/>
+        </geometry>
+        <material name="grey"/>
+    </visual>
+</link>
+<link name="shaftF">
+    <visual>
+        <origin xyz="0.0 0.0 0.009" rpy="1.57 0.0 0.0"/>
+        <geometry>
+            <mesh filename="${shaft}" scale= "${scale}"/>
+        </geometry>
+        <material name="grey"/>
+    </visual>
+</link>
+<link name="shaftB">
+    <visual>
+        <origin xyz="0.0 0.0 0.009" rpy="1.57 0.0 0.0"/>
+        <geometry>
+            <mesh filename="${shaft}" scale= "${scale}"/>
+        </geometry>
+        <material name="grey"/>
+    </visual>
+</link>
+<joint name="mainBody_shaftF" type="fixed">
+    <parent link="base_link"/>
+    <child link="shaftF"/>
+    <origin xyz="0.07 0 0.0105" rpy="0.0 0.0 0.0"/>
+</joint>
+<joint name="mainBody_shaftB" type="fixed">
+    <parent link="base_link"/>
+    <child link="shaftB"/>
+    <origin xyz="-0.07 0 0.0105" rpy="0.0 0.0 0.0"/>
+</joint>
 <joint name="mainBody_WheelBL" type="fixed">
     <parent link="base_link"/>
     <child link="wheelBL"/>
-    <origin xyz="-0.7 0.57 0.10" rpy="0.0 0.0 0.0"/>
+    <origin xyz="-0.07 0.0525 0.01" rpy="0.0 0.0 0.0"/>
+    <axis xyz="0 1 0"/>
+    <limit lower="0" upper="0" effort="0" velocity="0"/>
 </joint>
 <joint name="mainBody_WheelFL" type="fixed">
     <parent link="base_link"/>
     <child link="wheelFL"/>
-    <origin xyz="0.07 0.057 0.010" rpy="0.0 0.0 0.0"/>
+    <origin xyz="0.07 0.0525 0.010" rpy="0.0 0.0 0.0"/>
+    <axis xyz="0 1 0"/>
+    <limit lower="0" upper="0" effort="0" velocity="0"/>
 </joint>
 <joint name="mainBody_WheelFR" type="fixed">
     <parent link="base_link"/>
     <child link="wheelFR"/>
-    <origin xyz="0.07 -0.048 0.010" rpy="0.0 0.0 0.0"/>
+    <origin xyz="0.07 -0.0525 0.010" rpy="0.0 0.0 0.0"/>
+    <axis xyz="0 1 0"/>
+    <limit lower="0" upper="0" effort="0" velocity="0"/>
 </joint>
 <joint name="mainBody_WheelBR" type="fixed">
     <parent link="base_link"/>
     <child link="wheelBR"/>
-    <origin xyz="-0.07 -0.048 0.010" rpy="0.0 0.0 0.0"/>
+    <origin xyz="-0.07 -0.0525 0.010" rpy="0.0 0.0 0.0"/>
+    <axis xyz="0 1 0"/>
+    <limit lower="0" upper="0" effort="0" velocity="0"/>
+</joint>
+<joint name="mainBody_Lidar" type="fixed">
+    <parent link="base_link"/>
+    <child link="lidar"/>
+    <origin xyz="0.075 0 0.04" rpy="0.0 0.0 0.0"/>
 </joint>
 </robot>
